File: usb-magnetometer.kicad_pcb (KiCad board)
At the start: 4 copper layers, 59.4 x 19.8 mm, 44 parts, among them J1 USB_C_Receptacle_USB2.0, J2 1x5_MALE, J3 1x2_Male, J4 Conn_02x04_Odd_Even, J5 Conn_02x04_Odd_Even, J6 Conn_02x04_Odd_Even, J7 Conn_02x04_Odd_Even, U1 FT231XS, U2 TMAG5170, U3 STM32L010C6T6

Commit message: Make two pcb as one design
Parts:
- added REF**: CNSN_PanelTabPerforations_0.3mmx8, CNSN_DfX:CNSN_PanelTabPerforations_0.3mmx8, F.Cu at (96.8, 143.4)
- added REF**: CNSN_PanelTabPerforations_0.3mmx8, CNSN_DfX:CNSN_PanelTabPerforations_0.3mmx8, F.Cu at (93.8, 143.4)
- moved C9 0.10 mm to (101.4, 147.2)
- moved J6 0.10 mm to (98.4, 139.8)
- moved C11 0.10 mm to (99.8, 144.9)
- moved J4 0.10 mm to (103.0, 143.3)
- moved U2 0.10 mm to (102.1, 143.3)
Other:
- board size 59.4 x 19.8 mm -> 59.5 x 19.8 mm
